File: design_files/AST1001.sch (EAGLE design)
At the start: 6 parts, among them J1 SM05B, U1 BMA250

Commit message: updates
Parts:
- C2: value 10uF -> 1uF; device tinycircuits:AS-ITM-00002 -> tinycircuits:AS-ITM-00410; PARTNO (none) -> AS-ITM-00410; VALUE (none) -> 1uF
- J1: device tinycircuits:AS-ITM-00340 -> tinycircuits:AS-ITM-00340EDGE
- R1, R2: value 0.0 -> 1.00K; device tinycircuits:AS-ITM-00076 -> tinycircuits:AS-ITM-00003; PARTNO (none) -> AS-ITM-00003; VALUE (none) -> 1.00K
- U1: value BMA250 -> BMA250E
Other:
- note added: "BMA250 Accelerometer"
- note added: "Hand Populated: -"
- note added: "Hand Soldered: -"
- note added: "Non Populated: -"
- note added: "Notes: -"
- note added: "Variant: Standard - R"
- note added: "Wireling Accelerometer"
- note removed: "Accelerometer Sensor Board"
- note removed: "BMA250 Accelerometer Sensor"
